File: PCB/rgb_led.sch (KiCad schematic (older format))
At the start: 2 parts

Commit message: Schematic V2
REQUIRES CHANGE TO SOFTWARE: Changed pin of LAT from D7 to D0 to avoid
using the non-maskable interrupt pin.

Added a SMD LED D8 to provide and enviornmental lighting effect.

Removed power supply circuit; USB power from the dev board is sufficent
for
LED brightness. Must be plugged into USB 3.0 or a 2A rated supply.

Updated symbol library to use KiBOM and to Lib Version 4.

TODO: Update  PCB
Parts:
- C4: symbol Capacitor -> local:Capacitor; Config (none) -> Fit; Included in BOM Yes -> (none)
- D0: symbol LED_RGB_Common_Anode -> local:LED_RGB_Common_Anode; Config (none) -> Fit; Included in BOM Yes -> (none)
Changed lines of the file:
@@
-EESchema Schematic File Version 2
+EESchema Schematic File Version 4
 LIBS:local
 LIBS:Christmas_Tree_Disco-cache
@@
 $Descr A 11000 8500
 encoding utf-8
-Sheet 11 20
+Sheet 13 19
 Title "Christmas Tree Disco"
-Date "2017-09-10"
-Rev "V1.1"
+Date "2017-09-20"
+Rev "V2"
 Comp "www.GitHub.com/Cryochasm"
 Comment1 ""
@@
 $EndDescr
 $Comp
-L LED_RGB_Common_Anode D0
+L local:LED_RGB_Common_Anode D0
 U 1 1 5980D97F
 P 5400 3300
@@
 AR Path="/59809489/5980966C/598171EF/5980D97F" Ref="D11"  Part="1"
 AR Path="/59809489/5980966C/59837C41/5980D97F" Ref="D12"  Part="1"
-F 0 "D7" V 5354 3622 50  0000 L CNN
+F 0 "D12" V 5354 3622 50  0000 L CNN
 F 1 "RGB LED" V 5445 3622 50  0000 L CNN
 F 2 "local:T-1_5mm" H 5450 3300 60  0001 C CNN
@@
 F 4 " WP154A4SEJ3VBDZGW/CA" H 5400 3300 60  0001 C CNN "MPN"
 F 5 "Red, Green, Blue (RGB) 625nm Red, 525nm Green, 470nm Blue LED Indication - Discrete 2.2V Red, 3.3V Green, 3.3V Blue Radial" H 5400 3300 60  0001 C CNN "Description"
-F 6 "Yes" H 5400 3300 60  0001 C CNN "Included in BOM"
+F 6 "Fit" H 5400 3300 60  0001 C CNN "Config"
 	1    5400 3300
 	0    1    1    0
 $EndComp
 Wire Wire Line
-	5400 3000 5400 3200
+	5400 3000 5400 3100
 Text HLabel 1100 2900 0    50   Input ~ 0
 ~~RGB[0..2]
@@
 	1100 2400 1200 2400
 Wire Bus Line
-	1200 2400 1200 2600
-Wire Bus Line
 	1100 2900 1200 2900
-Wire Bus Line
-	1200 2900 1200 3200
 Entry Wire Line
 	1200 2500 1300 2600
@@
 GND
 $Comp
-L Capacitor C4
+L local:Capacitor C4
 U 1 1 59893093
 P 4600 3300
@@
 AR Path="/59809489/5980966C/59815DAA/59893093" Ref="C15"  Part="1"
 AR Path="/59809489/5980966C/598171EF/59893093" Ref="C11"  Part="1"
-F 0 "C7" V 4554 3368 50  0000 L CNN
+F 0 "C12" V 4554 3368 50  0000 L CNN
 F 1 "0.1u" V 4645 3368 50  0000 L CNN
 F 2 "local:SMD-0805" H 4600 3300 60  0001 C CNN
@@
 F 4 "CL21B104KACWPNC" H 4600 3300 60  0001 C CNN "MPN"
 F 5 "0.1µF ±10% 25V Ceramic Capacitor X7R 0805 (2012 Metric)" H 4600 3300 60  0001 C CNN "Description"
-F 6 "Yes" H 4600 3300 60  0001 C CNN "Included in BOM"
+F 6 "Fit" H 4600 3300 60  0001 C CNN "Config"
 	1    4600 3300
 	0    1    1    0
 $EndComp
+Wire Wire Line
+	5400 3100 5400 3200
+Wire Bus Line
+	1200 2400 1200 2600
+Wire Bus Line
+	1200 2900 1200 3200
 $EndSCHEMATC
