File: PCB/rgb_led_array.sch (KiCad schematic (older format))
At the start: 2 parts, among them U2 TLC5955DCA

Commit message: Footprint Modifications
Parts:
- C16: footprint local:SMD-POL-1206 -> local:SMD-TANT-1206
Changed lines of the file:
@@
 Sheet 4 20
 Title "Christmas Tree Disco"
-Date "2017-08-23"
-Rev "V1.0"
+Date "2017-09-10"
+Rev "V1.1"
 Comp "www.GitHub.com/Cryochasm"
 Comment1 ""
@@
 F 0 "C16" V 6500 1100 50  0000 R CNN
 F 1 "10u" V 6600 1000 50  0000 C CNN
-F 2 "local:SMD-POL-1206" H 6600 800 60  0001 C CNN
+F 2 "local:SMD-TANT-1206" H 6600 800 60  0001 C CNN
 F 3 "http://datasheets.avx.com/F93.pdf" H 6600 800 60  0001 C CNN
 F 4 "F931A106KAA" H 6600 800 60  0001 C CNN "MPN"

Commit message: Schematic V2
REQUIRES CHANGE TO SOFTWARE: Changed pin of LAT from D7 to D0 to avoid
using the non-maskable interrupt pin.

Added a SMD LED D8 to provide and enviornmental lighting effect.

Removed power supply circuit; USB power from the dev board is sufficent
for
LED brightness. Must be plugged into USB 3.0 or a 2A rated supply.

Updated symbol library to use KiBOM and to Lib Version 4.

TODO: Update  PCB
Parts:
- added C8: 0.1u, local:SMD-0805, symbol local:Capacitor
- added D8: AAA3528SEEZGKQBKS, local:PLCC-4-3.5x2.8, symbol local:LED_RGB_Common_Anode
- C16: symbol Capacitor-Pol -> local:Capacitor-Pol; Config (none) -> Fit; Included in BOM Yes -> (none)
- U2: symbol TLC5955DCA -> local:TLC5955DCA; Config (none) -> Fit; Included in BOM Yes -> (none)
Connections:
- net 5V: now also C8.1, D8.2 (CATHODE)
- net GND: now also C8.2
- net at U2.51 (OUTG8): now also D8.3 (BLU)
- net at U2.52 (OUTR8): now also D8.1 (RED)
- net at U2.53 (OUTB8): now also D8.4 (GRN)
- no-connect marks 3 -> 0
Other:
- moved on the sheet: C16, U2
